File: KiCAD Files/SiemensET200BExpansionBoard.kicad_pcb (KiCad board)
At the start: 2 copper layers, 85.1 x 50 mm, 39 parts, among them J1 Screw_Terminal_01x02, J2 Conn_01x16, SW1 SW_SPDT, SW10 SW_SPDT, SW11 SW_SPDT, SW12 SW_SPDT, SW13 SW_SPDT, SW14 SW_SPDT, SW15 SW_SPDT, SW16 SW_SPDT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

Commit message: Add qrcode
Parts:
- added G***: LOGO, Footprint:qrcode, B.Cu at (158.1, 121.4)
- moved G*** 25.3 mm to (158.1, 103.5)
Other:
- board text added: "JLCJLCJLCJLC"
